File: caretaker-device-dimmer/eagle/caretaker-dimmer.sch (EAGLE design)
At the start: 40 parts, among them IC1 LD33V, IC2 ATmega168-20PU, IC4 MOC3023M, Q1 16MHz, T1 BC547B

Commit message: feat: Update images, bump version
Other:
- note added: "3"
- note removed: "2"
Changed lines of the file:
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@@
 <plain>
 <text x="163.83" y="31.75" size="2.54" layer="94">Dirk Grappendorf</text>
-<text x="251.46" y="7.62" size="2.54" layer="94">2</text>
+<text x="251.46" y="7.62" size="2.54" layer="94">3</text>
 <text x="163.83" y="27.94" size="2.54" layer="94">grappendorf.net</text>
 <text x="163.83" y="24.13" size="2.54" layer="94">CERN Open Hardware License 1.1</text>
